Commit message: working code - with 4 inputs

File: urdf/milliampere.urdf.xacro (robot description, xacro)
@@ -7,5 +7,5 @@
   <link name="base_link">
   <visual>
-    <origin xyz="0 0 ${-draught + H/2.0}" rpy="0 0 0"/>
+    <origin xyz="0 0 ${-0.2 + H/2.0}" rpy="0 0 0"/> // 0.2m = draught
     <geometry>
       <box size="${L} ${W} ${H}"/>
@@ -16,5 +16,5 @@
   </visual>
   <collision>
-    <origin xyz="0 0 ${-draught + H/2.0}" rpy="0 0 0"/>
+    <origin xyz="0 0 ${-0.2 + H/2.0}" rpy="0 0 0"/>
     <geometry>
       <box size="${L} ${W} ${H}"/>
